File: SGTC/amplifier.kicad_sch (KiCad schematic)
At the start: 6 parts

Commit message: added schematic to new SGTC
Parts:
- removed R2, R3, R4: R_US, symbol Device:R_US
- removed U1: ~, Library:StrainGaugeGND, symbol My_Library:StrainGaugeGND
- removed U3: ~, Library:StrainGaugeV, symbol My_Library:StrainGaugeV
- added C7: 0.1 uF, Capacitor_SMD:C_0603_1608Metric, symbol Device:C_Small
- added C8: 10 uF, Capacitor_SMD:C_0805_2012Metric, symbol Device:C_Small
- added U5: AD8421, Package_SO:MSOP-8_3x3mm_P0.65mm, symbol Amplifier_Instrumentation:AD8421
- R1: value R_US -> 100; footprint (none) -> Resistor_SMD:R_0603_1608Metric
Connections:
- net +5V: now also C7.1, C8.1, U5.8 (Vs+)
- net GND: now also C7.2, C8.2, U5.5 (Vs-), U5.6 (Ref)
- net at R1.2: now also U5.3 (Rg)
- net A1_IN_P: no longer names the net of R1.1
- net A1_IN_P: now also U5.2 (Rg)
- new net A_IN_N: U5.1 (-)
- new net A_IN_P: U5.4 (+)
- new net A_OUT: U5.7
Other:
- note removed: "Fin Side 1 (Tension)"
- note removed: "comp"
- note removed: "tension"
