File: SGTC/StrainGauge.kicad_sch (KiCad schematic)
At the start: 6 parts

Commit message: strain gauge fix
Parts:
- removed R1, R2, R3, R4: R_US, symbol Device:R_US
- U3: footprint Library:StrainGaugeV -> Library:StrainGaugeGND
Connections:
- net +5V renamed +3.3V
Other:
- note removed: "comp"
- note removed: "tension"
