File: SGTC/StrainGauge2.kicad_sch (KiCad schematic)
At the start: 2 parts

Commit message: strain gauge fix
Connections:
- net +5V renamed +3.3V
Changed lines of the file:
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@@
 			)
 		)
-		(property "Value" "+5V"
+		(property "Value" "+3.3V"
 			(at 133.35 93.9799 90)
 			(effects
