File: teensy-breakout/teensy-breakout/teensy-breakout.kicad_sch (KiCad schematic)
At the start: 10 parts, among them J1 Conn_01x11_Pin, U1 Teensy4.1, U2 TPS62163DSGR, U3 LSM6DSO32TR

Commit message: routing go brrr
Parts:
- removed J1: Conn_01x11_Pin, symbol Connector:Conn_01x11_Pin
- added J1, J3: Conn_01x06_Pin, Connector_PinHeader_2.54mm:PinHeader_1x06_P2.54mm_Vertical, symbol Connector:Conn_01x06_Pin
- C1, C2: footprint (none) -> Capacitor_SMD:C_0805_2012Metric
- C3, C4: footprint (none) -> Capacitor_SMD:C_0603_1608Metric
- L1: footprint (none) -> teensy:LCXHF3030QKT2R2MNR
- R1: footprint (none) -> Resistor_SMD:R_0603_1608Metric
- U1: footprint (none) -> teensy:Teensy41
- U2: footprint DSG0008A -> teensy:TPS62163
- U3: footprint LGA-14L_2P5X3X0P83_STM -> teensy:LSM6DSO32
Connections:
- net +3.3V: now also C4.1, U1.46 (3V3), U3.5 (VDDIO), J1.5 (Pin_5)
- net ACLK: now also U1.29 (37_CS), J1.2 (Pin_2); no longer U1.9 (7_RX2_OUT1A)
- net CS_LSM: now also U1.28 (36_CS); no longer U1.24 (32_OUT1B)
- net GND: now also U1.1 (GND), U1.34 (GND), U1.47 (GND), U1.52 (GND), U1.58 (GND), U1.59 (GND), J1.6 (Pin_6)
- net INT1: no longer U3.9 (INT2)
- net INT2: now also U3.9 (INT2)
- net MISO: now also J1.3 (Pin_3)
- net MOSI: now also J3.5 (Pin_5)
- net SCLK: now also J3.6 (Pin_6)
- net VBAT: now also J1.1 (Pin_1)
- net ~{CS_1}: now also U1.4 (2_OUT2), J3.1 (Pin_1); no longer U1.5 (3_LRCLK2)
- net ~{CS_2}: now also U1.5 (3_LRCLK2), J3.2 (Pin_2); no longer U1.6 (4_BCLK2)
- net ~{CS_3}: now also U1.6 (4_BCLK2), J3.3 (Pin_3); no longer U1.7 (5_IN2)
- net ~{CS_4}: now also U1.7 (5_IN2), J3.4 (Pin_4); no longer U1.8 (6_OUT1D)
- net ~{DRDY}: now also U1.32 (40_A16), J1.4 (Pin_4); no longer U1.4 (2_OUT2)
- no-connect marks 0 -> 42
