File: Hardware/fin/fin.kicad_sch (KiCad schematic)
At the start: 44 parts, among them J1 Conn_01x07, J2 Conn_01x04_Pin, J3 Conn_01x04_Pin, J4 Conn_ARM_SWD_TagConnect_TC203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, J5 Conn_01x04_Pin, U1 ADS131M03QPWRQ1, U2 ADXL380-1BCCZ-RL7, U3 W25N512GVEIG, U4 TMP235A4DBZR, U5 STM32L412K8Ux, U6 ADXL380-1BCCZ-RL7, X1 ECS-327TXO-33-TR

Commit message: ground pours go brrrrrrrrrrrrrrrrr
Parts:
- J2, J3: footprint Connector_PinHeader_2.54mm:PinHeader_1x04_P2.54mm_Vertical -> Connector_PinHeader_2.54mm:PinHeader_2x02_P2.54mm_Vertical
Changed lines of the file:
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@@
 			)
 		)
-		(property "Footprint" "Connector_PinHeader_2.54mm:PinHeader_1x04_P2.54mm_Vertical"
+		(property "Footprint" "Connector_PinHeader_2.54mm:PinHeader_2x02_P2.54mm_Vertical"
 			(at 289.306 64.008 0)
 			(hide yes)
@@
 			)
 		)
-		(property "Footprint" "Connector_PinHeader_2.54mm:PinHeader_1x04_P2.54mm_Vertical"
+		(property "Footprint" "Connector_PinHeader_2.54mm:PinHeader_2x02_P2.54mm_Vertical"
 			(at 289.306 43.688 0)
 			(hide yes)

Commit message: add 1.65V ldo
Parts:
- added C6, C7: 1 uF, Capacitor_SMD:C_0402_1005Metric, symbol Device:C_Small
- added U7: ADP172ACBZ-1.65-R7, FinLib:CB-4-4_ADI, symbol FinLib:ADP172ACBZ-1.65-R7
Connections:
- net GAUGE2_IN_N is gone; now on net +1.65V: R13.2, R14.2, R4.2
- net +3.3V: now also C7.2, U7.A1 (VIN), U7.B1 (EN)
- net GND: now also C6.2, C7.1, U7.B2 (GND)
- net GAUGE1_IN_N renamed +1.65V
- net +1.65V: now also C6.1, U7.A2 (VOUT)
Other:
- moved on the sheet: U4
